File: electrical_schematic/kicad_procejt_FPV.kicad_sch (KiCad schematic)
At the start: 15 parts, among them J1 MPU-6050, J10 GPS BZ181, J11 NUCLEO - STM32L432KCU, J12 Conn_01x15_Pin, J13 LoRa, J14 LoRa, J2 BEC 12s, J3 BME280, J4 EM40A, J5 Conn_02x01, J6 Conn_01x02_Pin, J7 M3, J8 Conn_01x03_Pin, J9 DO_NUCELO

Commit message: Add files via upload
poprawioy sychamt spi i2c uart
Connections:
- net +3.3V: now also J12.14 (Pin_14); no longer J12.13 (Pin_13)
- net +5V: now also J12.4 (Pin_4), J2.1 (Pin_1)
Other:
- note added: "A8 A0 A1 A2 A3"
- note added: "uart"
- note removed: "A3 A2 A7 A1 A0"
Changed lines of the file:
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@@
+		)
+	)
+	(text "uart\n"
+		(exclude_from_sim no)
+		(at 138.684 64.77 0)
+		(effects
+			(font
+				(size 1.27 1.27)
+			)
 		)
 	)
@@
 		)
 	)
-	(text "A3\nA2\nA7\nA1\nA0\n\n"
+	(text "A8\nA0\nA1\nA2\nA3\n\n"
 		(exclude_from_sim no)
 		(at 128.524 145.034 0)
@@
 	)
 	(junction
+		(at 182.88 74.93)
+		(diameter 0)
+		(color 0 0 0 0)
+	)
+	(junction
 		(at 176.53 113.03)
 		(diameter 0)
@@
 	(wire
 		(pts
+			(xy 179.07 100.33) (xy 179.07 97.79)
+		)
+		(stroke
+			(width 0)
+			(type default)
+		)
+	)
+	(wire
+		(pts
 			(xy 82.55 78.74) (xy 125.73 78.74)
 		)
@@
 	(wire
 		(pts
+			(xy 171.45 100.33) (xy 179.07 100.33)
+		)
+		(stroke
+			(width 0)
+			(type default)
+		)
+	)
+	(wire
+		(pts
 			(xy 114.3 39.37) (xy 114.3 41.91)
 		)
@@
 	(wire
 		(pts
-			(xy 171.45 74.93) (xy 187.96 74.93)
+			(xy 171.45 74.93) (xy 182.88 74.93)
 		)
 		(stroke
@@
 	(wire
 		(pts
+			(xy 182.88 76.2) (xy 182.88 74.93)
+		)
+		(stroke
+			(width 0)
+			(type default)
+		)
+	)
+	(wire
+		(pts
 			(xy 163.83 132.08) (xy 129.54 132.08)
 		)
@@
 	(wire
 		(pts
+			(xy 182.88 74.93) (xy 187.96 74.93)
+		)
+		(stroke
+			(width 0)
+			(type default)
+		)
+	)
+	(wire
+		(pts
 			(xy 133.35 134.62) (xy 163.83 134.62)
 		)
@@
 	(wire
 		(pts
+			(xy 181.61 76.2) (xy 182.88 76.2)
+		)
+		(stroke
+			(width 0)
+			(type default)
+		)
+	)
+	(wire
+		(pts
 			(xy 118.11 100.33) (xy 111.76 100.33)
 		)
@@
 		)
 		(stroke
-			(width 0)
-			(type default)
-		)
-	)
-	(wire
-		(pts
-			(xy 171.45 97.79) (xy 179.07 97.79)
-		)
-		(stroke
